File: PCB/Pack/Pack.sch (KiCad schematic (older format))
At the start: 77 parts, among them J1 Conn_01x01, J2 Conn_01x01, J3 Conn_01x01, J4 Conn_01x01, J5 Conn_01x01, J6 Conn_01x01, J7 Conn_01x02, J8 Conn_01x02

Commit message: minor stuff
Parts:
- LOGO1: renamed from LOGO?; footprint ENNOID:ENNOID-LOGO -> (none)
Changed lines of the file:
@@
 	1550 1600 1550 1300
 $Comp
-L Graphic:Logo_Open_Hardware_Small LOGO?
+L Graphic:Logo_Open_Hardware_Small LOGO1
 U 1 1 5C700030
 P 7500 6850
-F 0 "LOGO?" H 7500 7125 50  0001 C CNN
+F 0 "LOGO1" H 7500 7125 50  0001 C CNN
 F 1 "Logo_Open_Hardware_Small" H 7500 6625 50  0001 C CNN
-F 2 "ENNOID:ENNOID-LOGO" H 7500 6850 50  0001 C CNN
+F 2 "" H 7500 6850 50  0001 C CNN
 F 3 "~" H 7500 6850 50  0001 C CNN
 	1    7500 6850
 	1    0    0    -1
 $EndComp
+Wire Notes Line
+	1900 850  1900 5750
+Wire Notes Line
+	1900 5750 1250 5750
+Wire Notes Line
+	1250 5750 1250 850
+Wire Notes Line
+	1250 850  1900 850
 $EndSCHEMATC

Commit message: gerber
Parts:
- F1, F2, F3: footprint Fuse_Holders_and_Fuses:Fuse_SMD1206_Wave -> (none)
Changed lines of the file:
@@
 F 0 "F3" H 1610 4496 50  0000 L CNN
 F 1 "Fuse" H 1610 4405 50  0000 L CNN
-F 2 "Fuse_Holders_and_Fuses:Fuse_SMD1206_Wave" V 1480 4450 50  0001 C CNN
+F 2 "" V 1480 4450 50  0001 C CNN
 F 3 "~" H 1550 4450 50  0001 C CNN
 	1    1550 4450
@@
 F 0 "F2" H 1610 2946 50  0000 L CNN
 F 1 "Fuse" H 1610 2855 50  0000 L CNN
-F 2 "Fuse_Holders_and_Fuses:Fuse_SMD1206_Wave" V 1480 2900 50  0001 C CNN
+F 2 "" V 1480 2900 50  0001 C CNN
 F 3 "~" H 1550 2900 50  0001 C CNN
 	1    1550 2900
@@
 F 0 "F1" H 1610 1796 50  0000 L CNN
 F 1 "Fuse" H 1610 1705 50  0000 L CNN
-F 2 "Fuse_Holders_and_Fuses:Fuse_SMD1206_Wave" V 1480 1750 50  0001 C CNN
+F 2 "" V 1480 1750 50  0001 C CNN
 F 3 "~" H 1550 1750 50  0001 C CNN
 	1    1550 1750

Commit message: no more on board fuses
Parts:
- removed F1, F2, F3: Fuse, symbol Device:Fuse
- removed F10, F11, F12, F13, F14, F15, F16, F17, F18, F19, F20, F21, F22, F23, F24, F25, F26, F27, F28, F29, F30, F31, F32, F33, F4, F5, F6, F7, F8, F9: Fuse, Fuse_Holders_and_Fuses:Fuse_SMD1206_Wave, symbol Device:Fuse
Connections:
- wire segments 152 -> 119

Commit message: small change
Parts:
- BT1, BT10, BT11, BT12, BT13, BT14, BT15, BT16, BT17, BT18, BT19, BT2, BT20, BT21, BT22, BT23, BT24, BT25, BT26, BT27, BT28, BT29, BT3, BT30, BT4, BT5, BT6, BT7, BT8, BT9: footprint ENNOID:Battery -> ENNOID:18650
Changed lines of the file:
@@
 F 0 "BT1" H 2418 2396 50  0000 L CNN
 F 1 "Battery_Cell" H 2418 2305 50  0000 L CNN
-F 2 "ENNOID:Battery" V 2300 2360 50  0001 C CNN
+F 2 "ENNOID:18650" V 2300 2360 50  0001 C CNN
 F 3 "~" V 2300 2360 50  0001 C CNN
 	1    2300 2300
@@
 F 0 "BT4" H 3118 2396 50  0000 L CNN
 F 1 "Battery_Cell" H 3118 2305 50  0000 L CNN
-F 2 "ENNOID:Battery" V 3000 2360 50  0001 C CNN
+F 2 "ENNOID:18650" V 3000 2360 50  0001 C CNN
 F 3 "~" V 3000 2360 50  0001 C CNN
 	1    3000 2300
@@
 F 0 "BT7" H 3868 2396 50  0000 L CNN
 F 1 "Battery_Cell" H 3868 2305 50  0000 L CNN
-F 2 "ENNOID:Battery" V 3750 2360 50  0001 C CNN
+F 2 "ENNOID:18650" V 3750 2360 50  0001 C CNN
 F 3 "~" V 3750 2360 50  0001 C CNN
 	1    3750 2300
@@
 F 0 "BT10" H 4668 2396 50  0000 L CNN
 F 1 "Battery_Cell" H 4668 2305 50  0000 L CNN
-F 2 "ENNOID:Battery" V 4550 2360 50  0001 C CNN
+F 2 "ENNOID:18650" V 4550 2360 50  0001 C CNN
 F 3 "~" V 4550 2360 50  0001 C CNN
 	1    4550 2300
@@
 F 0 "BT13" H 5418 2396 50  0000 L CNN
 F 1 "Battery_Cell" H 5418 2305 50  0000 L CNN
-F 2 "ENNOID:Battery" V 5300 2360 50  0001 C CNN
+F 2 "ENNOID:18650" V 5300 2360 50  0001 C CNN
 F 3 "~" V 5300 2360 50  0001 C CNN
 	1    5300 2300
@@
 F 0 "BT16" H 6118 2396 50  0000 L CNN
 F 1 "Battery_Cell" H 6118 2305 50  0000 L CNN
-F 2 "ENNOID:Battery" V 6000 2360 50  0001 C CNN
+F 2 "ENNOID:18650" V 6000 2360 50  0001 C CNN
 F 3 "~" V 6000 2360 50  0001 C CNN
 	1    6000 2300
@@
 F 0 "BT19" H 6818 2396 50  0000 L CNN
 F 1 "Battery_Cell" H 6818 2305 50  0000 L CNN
-F 2 "ENNOID:Battery" V 6700 2360 50  0001 C CNN
+F 2 "ENNOID:18650" V 6700 2360 50  0001 C CNN
 F 3 "~" V 6700 2360 50  0001 C CNN
 	1    6700 2300
@@
 F 0 "BT22" H 7518 2396 50  0000 L CNN
 F 1 "Battery_Cell" H 7518 2305 50  0000 L CNN
-F 2 "ENNOID:Battery" V 7400 2360 50  0001 C CNN
+F 2 "ENNOID:18650" V 7400 2360 50  0001 C CNN
 F 3 "~" V 7400 2360 50  0001 C CNN
 	1    7400 2300
@@
 F 0 "BT25" H 8218 2396 50  0000 L CNN
 F 1 "Battery_Cell" H 8218 2305 50  0000 L CNN
-F 2 "ENNOID:Battery" V 8100 2360 50  0001 C CNN
+F 2 "ENNOID:18650" V 8100 2360 50  0001 C CNN
 F 3 "~" V 8100 2360 50  0001 C CNN
 	1    8100 2300
@@
 F 0 "BT28" H 8918 2396 50  0000 L CNN
 F 1 "Battery_Cell" H 8918 2305 50  0000 L CNN
-F 2 "ENNOID:Battery" V 8800 2360 50  0001 C CNN
+F 2 "ENNOID:18650" V 8800 2360 50  0001 C CNN
 F 3 "~" V 8800 2360 50  0001 C CNN
 	1    8800 2300
@@
 F 0 "BT2" H 2418 3546 50  0000 L CNN
 F 1 "Battery_Cell" H 2418 3455 50  0000 L CNN
-F 2 "ENNOID:Battery" V 2300 3510 50  0001 C CNN
+F 2 "ENNOID:18650" V 2300 3510 50  0001 C CNN
 F 3 "~" V 2300 3510 50  0001 C CNN
 	1    2300 3450
@@
 F 0 "BT5" H 3118 3546 50  0000 L CNN
 F 1 "Battery_Cell" H 3118 3455 50  0000 L CNN
-F 2 "ENNOID:Battery" V 3000 3510 50  0001 C CNN
+F 2 "ENNOID:18650" V 3000 3510 50  0001 C CNN
 F 3 "~" V 3000 3510 50  0001 C CNN
 	1    3000 3450
@@
 F 0 "BT8" H 3868 3546 50  0000 L CNN
 F 1 "Battery_Cell" H 3868 3455 50  0000 L CNN
-F 2 "ENNOID:Battery" V 3750 3510 50  0001 C CNN
+F 2 "ENNOID:18650" V 3750 3510 50  0001 C CNN
 F 3 "~" V 3750 3510 50  0001 C CNN
 	1    3750 3450
@@
 F 0 "BT11" H 4668 3546 50  0000 L CNN
 F 1 "Battery_Cell" H 4668 3455 50  0000 L CNN
-F 2 "ENNOID:Battery" V 4550 3510 50  0001 C CNN
+F 2 "ENNOID:18650" V 4550 3510 50  0001 C CNN
 F 3 "~" V 4550 3510 50  0001 C CNN
 	1    4550 3450
@@
 F 0 "BT14" H 5418 3546 50  0000 L CNN
 F 1 "Battery_Cell" H 5418 3455 50  0000 L CNN
-F 2 "ENNOID:Battery" V 5300 3510 50  0001 C CNN
+F 2 "ENNOID:18650" V 5300 3510 50  0001 C CNN
 F 3 "~" V 5300 3510 50  0001 C CNN
 	1    5300 3450
@@
 F 0 "BT17" H 6118 3546 50  0000 L CNN
 F 1 "Battery_Cell" H 6118 3455 50  0000 L CNN
-F 2 "ENNOID:Battery" V 6000 3510 50  0001 C CNN
+F 2 "ENNOID:18650" V 6000 3510 50  0001 C CNN
 F 3 "~" V 6000 3510 50  0001 C CNN
 	1    6000 3450
@@
 F 0 "BT20" H 6818 3546 50  0000 L CNN
 F 1 "Battery_Cell" H 6818 3455 50  0000 L CNN
-F 2 "ENNOID:Battery" V 6700 3510 50  0001 C CNN
+F 2 "ENNOID:18650" V 6700 3510 50  0001 C CNN
 F 3 "~" V 6700 3510 50  0001 C CNN
 	1    6700 3450
@@
 F 0 "BT23" H 7518 3546 50  0000 L CNN
 F 1 "Battery_Cell" H 7518 3455 50  0000 L CNN
-F 2 "ENNOID:Battery" V 7400 3510 50  0001 C CNN
+F 2 "ENNOID:18650" V 7400 3510 50  0001 C CNN
 F 3 "~" V 7400 3510 50  0001 C CNN
 	1    7400 3450
@@
 F 0 "BT26" H 8218 3546 50  0000 L CNN
 F 1 "Battery_Cell" H 8218 3455 50  0000 L CNN
-F 2 "ENNOID:Battery" V 8100 3510 50  0001 C CNN
+F 2 "ENNOID:18650" V 8100 3510 50  0001 C CNN
 F 3 "~" V 8100 3510 50  0001 C CNN
 	1    8100 3450
@@
 F 0 "BT29" H 8918 3546 50  0000 L CNN
 F 1 "Battery_Cell" H 8918 3455 50  0000 L CNN
-F 2 "ENNOID:Battery" V 8800 3510 50  0001 C CNN
+F 2 "ENNOID:18650" V 8800 3510 50  0001 C CNN
 F 3 "~" V 8800 3510 50  0001 C CNN
 	1    8800 3450
@@
 F 0 "BT3" H 2418 5096 50  0000 L CNN
 F 1 "Battery_Cell" H 2418 5005 50  0000 L CNN
-F 2 "ENNOID:Battery" V 2300 5060 50  0001 C CNN
+F 2 "ENNOID:18650" V 2300 5060 50  0001 C CNN
 F 3 "~" V 2300 5060 50  0001 C CNN
 	1    2300 5000
@@
 F 0 "BT6" H 3118 5096 50  0000 L CNN
 F 1 "Battery_Cell" H 3118 5005 50  0000 L CNN
-F 2 "ENNOID:Battery" V 3000 5060 50  0001 C CNN
+F 2 "ENNOID:18650" V 3000 5060 50  0001 C CNN
 F 3 "~" V 3000 5060 50  0001 C CNN
 	1    3000 5000
@@
 F 0 "BT9" H 3868 5096 50  0000 L CNN
 F 1 "Battery_Cell" H 3868 5005 50  0000 L CNN
-F 2 "ENNOID:Battery" V 3750 5060 50  0001 C CNN
+F 2 "ENNOID:18650" V 3750 5060 50  0001 C CNN
 F 3 "~" V 3750 5060 50  0001 C CNN
 	1    3750 5000
@@
 F 0 "BT12" H 4668 5046 50  0000 L CNN
 F 1 "Battery_Cell" H 4668 4955 50  0000 L CNN
-F 2 "ENNOID:Battery" V 4550 5010 50  0001 C CNN
+F 2 "ENNOID:18650" V 4550 5010 50  0001 C CNN
 F 3 "~" V 4550 5010 50  0001 C CNN
 	1    4550 4950
@@
 F 0 "BT15" H 5418 5046 50  0000 L CNN
 F 1 "Battery_Cell" H 5418 4955 50  0000 L CNN
-F 2 "ENNOID:Battery" V 5300 5010 50  0001 C CNN
+F 2 "ENNOID:18650" V 5300 5010 50  0001 C CNN
 F 3 "~" V 5300 5010 50  0001 C CNN
 	1    5300 4950
@@
 F 0 "BT18" H 6118 5046 50  0000 L CNN
 F 1 "Battery_Cell" H 6118 4955 50  0000 L CNN
-F 2 "ENNOID:Battery" V 6000 5010 50  0001 C CNN
+F 2 "ENNOID:18650" V 6000 5010 50  0001 C CNN
 F 3 "~" V 6000 5010 50  0001 C CNN
 	1    6000 4950
@@
 F 0 "BT21" H 6818 5046 50  0000 L CNN
 F 1 "Battery_Cell" H 6818 4955 50  0000 L CNN
-F 2 "ENNOID:Battery" V 6700 5010 50  0001 C CNN
+F 2 "ENNOID:18650" V 6700 5010 50  0001 C CNN
 F 3 "~" V 6700 5010 50  0001 C CNN
 	1    6700 4950
@@
 F 0 "BT24" H 7518 5046 50  0000 L CNN
 F 1 "Battery_Cell" H 7518 4955 50  0000 L CNN
-F 2 "ENNOID:Battery" V 7400 5010 50  0001 C CNN
+F 2 "ENNOID:18650" V 7400 5010 50  0001 C CNN
 F 3 "~" V 7400 5010 50  0001 C CNN
 	1    7400 4950
@@
 F 0 "BT27" H 8218 5046 50  0000 L CNN
 F 1 "Battery_Cell" H 8218 4955 50  0000 L CNN
-F 2 "ENNOID:Battery" V 8100 5010 50  0001 C CNN
+F 2 "ENNOID:18650" V 8100 5010 50  0001 C CNN
 F 3 "~" V 8100 5010 50  0001 C CNN
 	1    8100 4950
@@
 F 0 "BT30" H 8918 5046 50  0000 L CNN
 F 1 "Battery_Cell" H 8918 4955 50  0000 L CNN
-F 2 "ENNOID:Battery" V 8800 5010 50  0001 C CNN
+F 2 "ENNOID:18650" V 8800 5010 50  0001 C CNN
 F 3 "~" V 8800 5010 50  0001 C CNN
 	1    8800 4950

Commit message: PCB major changes
Parts:
- added J9: Conn_01x02, Pin_Headers:Pin_Header_Straight_1x02_Pitch2.54mm_SMD_Pin1Left, symbol Connector_Generic:Conn_01x02
- added TH2: Thermistor, Resistors_SMD:R_0805_HandSoldering, symbol Device:Thermistor
- BT31, BT32, BT33: footprint ENNOID:Battery -> ENNOID:18650
- J7, J8: footprint Pin_Headers:Pin_Header_Straight_1x02_Pitch2.54mm -> Pin_Headers:Pin_Header_Straight_1x02_Pitch2.54mm_SMD_Pin1Left
- TH1, TH3: footprint Resistors_THT:R_Axial_DIN0309_L9.0mm_D3.2mm_P5.08mm_Vertical -> Resistors_SMD:R_0805_HandSoldering
Connections:
- new net: J9.1 (Pin_1), TH2.1
- new net: J9.2 (Pin_2), TH2.2
Changed lines of the file:
@@
 F 0 "BT31" H 1668 2396 50  0000 L CNN
 F 1 "Battery_Cell" H 1668 2305 50  0000 L CNN
-F 2 "ENNOID:Battery" V 1550 2360 50  0001 C CNN
+F 2 "ENNOID:18650" V 1550 2360 50  0001 C CNN
 F 3 "~" V 1550 2360 50  0001 C CNN
 	1    1550 2300
@@
 F 0 "BT32" H 1668 3546 50  0000 L CNN
 F 1 "Battery_Cell" H 1668 3455 50  0000 L CNN
-F 2 "ENNOID:Battery" V 1550 3510 50  0001 C CNN
+F 2 "ENNOID:18650" V 1550 3510 50  0001 C CNN
 F 3 "~" V 1550 3510 50  0001 C CNN
 	1    1550 3450
@@
 F 0 "BT33" H 1668 5096 50  0000 L CNN
 F 1 "Battery_Cell" H 1668 5005 50  0000 L CNN
-F 2 "ENNOID:Battery" V 1550 5060 50  0001 C CNN
+F 2 "ENNOID:18650" V 1550 5060 50  0001 C CNN
 F 3 "~" V 1550 5060 50  0001 C CNN
 	1    1550 5000
@@
 F 0 "TH1" V 9558 2600 50  0000 C CNN
 F 1 "Thermistor" V 9649 2600 50  0000 C CNN
-F 2 "Resistors_THT:R_Axial_DIN0309_L9.0mm_D3.2mm_P5.08mm_Vertical" H 9800 2600 50  0001 C CNN
+F 2 "Resistors_SMD:R_0805_HandSoldering" H 9800 2600 50  0001 C CNN
 F 3 "~" H 9800 2600 50  0001 C CNN
 	1    9800 2600
@@
 F 0 "TH3" V 9558 2950 50  0000 C CNN
 F 1 "Thermistor" V 9649 2950 50  0000 C CNN
-F 2 "Resistors_THT:R_Axial_DIN0309_L9.0mm_D3.2mm_P5.08mm_Vertical" H 9800 2950 50  0001 C CNN
+F 2 "Resistors_SMD:R_0805_HandSoldering" H 9800 2950 50  0001 C CNN
 F 3 "~" H 9800 2950 50  0001 C CNN
 	1    9800 2950
@@
 F 0 "J7" H 10730 2592 50  0000 L CNN
 F 1 "Conn_01x02" H 10730 2501 50  0000 L CNN
-F 2 "Pin_Headers:Pin_Header_Straight_1x02_Pitch2.54mm" H 10650 2600 50  0001 C CNN
+F 2 "Pin_Headers:Pin_Header_Straight_1x02_Pitch2.54mm_SMD_Pin1Left" H 10650 2600 50  0001 C CNN
 F 3 "~" H 10650 2600 50  0001 C CNN
 	1    10650 2600
@@
 F 0 "J8" H 10730 2942 50  0000 L CNN
 F 1 "Conn_01x02" H 10730 2851 50  0000 L CNN
-F 2 "Pin_Headers:Pin_Header_Straight_1x02_Pitch2.54mm" H 10650 2950 50  0001 C CNN
+F 2 "Pin_Headers:Pin_Header_Straight_1x02_Pitch2.54mm_SMD_Pin1Left" H 10650 2950 50  0001 C CNN
 F 3 "~" H 10650 2950 50  0001 C CNN
 	1    10650 2950
@@
 Wire Wire Line
 	1550 3850 1550 4800
+$Comp
+L Device:Thermistor TH2
+U 1 1 5C8376E2
+P 9800 3350
+F 0 "TH2" V 9558 3350 50  0000 C CNN
+F 1 "Thermistor" V 9649 3350 50  0000 C CNN
+F 2 "Resistors_SMD:R_0805_HandSoldering" H 9800 3350 50  0001 C CNN
+F 3 "~" H 9800 3350 50  0001 C CNN
+	1    9800 3350
+	0    1    1    0
+$EndComp
+Wire Wire Line
+	10000 3350 10450 3350
+$Comp
+L Connector_Generic:Conn_01x02 J9
+U 1 1 5C8376ED
+P 10650 3350
+F 0 "J9" H 10730 3342 50  0000 L CNN
+F 1 "Conn_01x02" H 10730 3251 50  0000 L CNN
+F 2 "Pin_Headers:Pin_Header_Straight_1x02_Pitch2.54mm_SMD_Pin1Left" H 10650 3350 50  0001 C CNN
+F 3 "~" H 10650 3350 50  0001 C CNN
+	1    10650 3350
+	1    0    0    -1
+$EndComp
+Wire Wire Line
+	10450 3450 9600 3450
+Wire Wire Line
+	9600 3450 9600 3350
 $EndSCHEMATC

Commit message: Final version
Parts:
- BT28, BT29, BT30, BT31, BT32, BT33: footprint ENNOID:18650 -> ENNOID:half
Changed lines of the file:
@@
 F 0 "BT28" H 8918 2396 50  0000 L CNN
 F 1 "Battery_Cell" H 8918 2305 50  0000 L CNN
-F 2 "ENNOID:18650" V 8800 2360 50  0001 C CNN
+F 2 "ENNOID:half" V 8800 2360 50  0001 C CNN
 F 3 "~" V 8800 2360 50  0001 C CNN
 	1    8800 2300
@@
 F 0 "BT29" H 8918 3546 50  0000 L CNN
 F 1 "Battery_Cell" H 8918 3455 50  0000 L CNN
-F 2 "ENNOID:18650" V 8800 3510 50  0001 C CNN
+F 2 "ENNOID:half" V 8800 3510 50  0001 C CNN
 F 3 "~" V 8800 3510 50  0001 C CNN
 	1    8800 3450
@@
 F 0 "BT30" H 8918 5046 50  0000 L CNN
 F 1 "Battery_Cell" H 8918 4955 50  0000 L CNN
-F 2 "ENNOID:18650" V 8800 5010 50  0001 C CNN
+F 2 "ENNOID:half" V 8800 5010 50  0001 C CNN
 F 3 "~" V 8800 5010 50  0001 C CNN
 	1    8800 4950
@@
 F 0 "BT31" H 1668 2396 50  0000 L CNN
 F 1 "Battery_Cell" H 1668 2305 50  0000 L CNN
-F 2 "ENNOID:18650" V 1550 2360 50  0001 C CNN
+F 2 "ENNOID:half" V 1550 2360 50  0001 C CNN
 F 3 "~" V 1550 2360 50  0001 C CNN
 	1    1550 2300
@@
 F 0 "BT32" H 1668 3546 50  0000 L CNN
 F 1 "Battery_Cell" H 1668 3455 50  0000 L CNN
-F 2 "ENNOID:18650" V 1550 3510 50  0001 C CNN
+F 2 "ENNOID:half" V 1550 3510 50  0001 C CNN
 F 3 "~" V 1550 3510 50  0001 C CNN
 	1    1550 3450
@@
 F 0 "BT33" H 1668 5096 50  0000 L CNN
 F 1 "Battery_Cell" H 1668 5005 50  0000 L CNN
-F 2 "ENNOID:18650" V 1550 5060 50  0001 C CNN
+F 2 "ENNOID:half" V 1550 5060 50  0001 C CNN
 F 3 "~" V 1550 5060 50  0001 C CNN
 	1    1550 5000

Commit message: Major update 12S10P
3dprintable casing for 12S10P 1.5kWh
Parts:
- removed J1, J2, J3, J4: Conn_01x01, Pin_Headers:Pin_Header_Straight_1x01_Pitch2.54mm, symbol Connector_Generic:Conn_01x01
- removed J7, J8, J9: Conn_01x02, Pin_Headers:Pin_Header_Straight_1x02_Pitch2.54mm_SMD_Pin1Left, symbol Connector_Generic:Conn_01x02
- added BT1, BT100, BT101, BT102, BT103, BT104, BT105, BT109, BT110, BT111, BT112, BT113, BT114, BT115, BT116, BT117, BT13, BT14, BT15, BT16, BT17, BT18, BT19, BT2, BT20, BT21, BT25, BT26, BT27, BT28, BT29, BT3, BT30, BT37, BT38, BT39, BT4, BT40, BT41, BT42, BT43, BT44, BT45, BT49, BT5, BT50, BT51, BT52, BT53, BT54, BT55, BT56, BT57, BT6, BT61, BT62, BT63, BT64, BT65, BT66, BT67, BT68, BT69, BT7, BT73, BT74, BT75, BT76, BT77, BT78, BT79, BT8, BT80, BT81, BT85, BT86, BT87, BT88, BT89, BT9, BT90, BT91, BT92, BT93, BT97, BT98, BT99: Battery_Cell, ENNOID:18650, symbol Device:Battery_Cell
- added J1, J3: Conn_01x13, Pin_Headers:Pin_Header_Straight_1x13_Pitch2.54mm, symbol Connector_Generic:Conn_01x13
- added J2: Conn_01x10, Pin_Headers:Pin_Header_Straight_1x10_Pitch2.54mm, symbol Connector_Generic:Conn_01x10
- added TH1, TH2: Thermistor, Resistors_SMD:R_0805_HandSoldering, symbol Device:Thermistor
- BT118: renamed from BT28; footprint ENNOID:half -> ENNOID:18650
- BT119: renamed from BT29; footprint ENNOID:half -> ENNOID:18650
- BT120: renamed from BT30; footprint ENNOID:half -> ENNOID:18650
- BT31, BT32, BT33: footprint ENNOID:half -> ENNOID:18650
- LOGO1: footprint (none) -> ENNOID:ENNOID-LOGO
- renumbered BT1 to BT10, BT25 to BT106, BT26 to BT107, BT27 to BT108, BT2 to BT11, BT3 to BT12, BT4 to BT22, BT5 to BT23, BT6 to BT24, BT7 to BT34, BT8 to BT35, BT9 to BT36, BT10 to BT46, BT11 to BT47, BT12 to BT48, BT13 to BT58, BT14 to BT59, BT15 to BT60, BT16 to BT70, BT17 to BT71, BT18 to BT72, BT19 to BT82, BT20 to BT83, BT21 to BT84, BT22 to BT94, BT23 to BT95, BT24 to BT96, J5 to J14, J6 to J15, TH1 to TH3, TH3 to TH4, TH2 to TH5
Connections:
- net at BT10.1 (+), BT106.1 (+), BT118.1 (+)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: now also BT33.2 (-), BT105.2 (-), BT117.2 (-), BT21.2 (-), BT45.2 (-), BT57.2 (-), BT69.2 (-), BT81.2 (-), BT9.2 (-), BT93.2 (-), J1.4 (Pin_4), J3.10 (Pin_10); no longer BT31.1 (+), J14.1 (Pin_1)
- net at BT10.2 (-), BT106.2 (-), BT107.1 (+)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: now also J1.3 (Pin_3), J3.11 (Pin_11); no longer BT31.2 (-), BT32.1 (+)
- net at BT107.2 (-), BT108.1 (+), BT11.2 (-)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: now also J1.2 (Pin_2), J3.12 (Pin_12); no longer BT32.2 (-), BT33.1 (+)
- net at BT108.2 (-), BT12.2 (-), BT120.2 (-)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: now also J1.1 (Pin_1), J3.13 (Pin_13); no longer BT33.2 (-)
- net at TH3.1: now also J2.5 (Pin_5)
- net at TH3.2: now also J2.6 (Pin_6)
- net at TH4.1: now also J2.7 (Pin_7)
- net at TH4.2: now also J2.8 (Pin_8)
- net at TH5.1: now also J2.9 (Pin_9)
- net at TH5.2: now also J2.10 (Pin_10)
- new net: BT1.1 (+), BT109.1 (+), BT13.1 (+), BT25.1 (+), BT37.1 (+), BT49.1 (+), BT61.1 (+), BT73.1 (+), BT85.1 (+), BT97.1 (+), J1.13 (Pin_13), J14.1 (Pin_1), J3.1 (Pin_1)
- new net: J2.1 (Pin_1), TH1.1
- new net: J2.2 (Pin_2), TH1.2
- new net: J2.3 (Pin_3), TH2.1
- new net: J2.4 (Pin_4), TH2.2
- new net: BT100.1 (+), BT111.2 (-), BT112.1 (+), BT15.2 (-), BT16.1 (+), BT27.2 (-), BT28.1 (+), BT3.2 (-), BT39.2 (-), BT4.1 (+), BT40.1 (+), BT51.2 (-), BT52.1 (+), BT63.2 (-), BT64.1 (+), BT75.2 (-), BT76.1 (+), BT87.2 (-), BT88.1 (+), BT99.2 (-), J1.10 (Pin_10), J3.4 (Pin_4)
- new net: BT110.2 (-), BT111.1 (+), BT14.2 (-), BT15.1 (+), BT2.2 (-), BT26.2 (-), BT27.1 (+), BT3.1 (+), BT38.2 (-), BT39.1 (+), BT50.2 (-), BT51.1 (+), BT62.2 (-), BT63.1 (+), BT74.2 (-), BT75.1 (+), BT86.2 (-), BT87.1 (+), BT98.2 (-), BT99.1 (+), J1.11 (Pin_11), J3.3 (Pin_3)
- new net: BT1.2 (-), BT109.2 (-), BT110.1 (+), BT13.2 (-), BT14.1 (+), BT2.1 (+), BT25.2 (-), BT26.1 (+), BT37.2 (-), BT38.1 (+), BT49.2 (-), BT50.1 (+), BT61.2 (-), BT62.1 (+), BT73.2 (-), BT74.1 (+), BT85.2 (-), BT86.1 (+), BT97.2 (-), BT98.1 (+), J1.12 (Pin_12), J3.2 (Pin_2)
- new net: BT104.2 (-), BT105.1 (+), BT116.2 (-), BT117.1 (+), BT20.2 (-), BT21.1 (+), BT32.2 (-), BT33.1 (+), BT44.2 (-), BT45.1 (+), BT56.2 (-), BT57.1 (+), BT68.2 (-), BT69.1 (+), BT8.2 (-), BT80.2 (-), BT81.1 (+), BT9.1 (+), BT92.2 (-), BT93.1 (+), J1.5 (Pin_5), J3.9 (Pin_9)
- new net: BT103.2 (-), BT104.1 (+), BT115.2 (-), BT116.1 (+), BT19.2 (-), BT20.1 (+), BT31.2 (-), BT32.1 (+), BT43.2 (-), BT44.1 (+), BT55.2 (-), BT56.1 (+), BT67.2 (-), BT68.1 (+), BT7.2 (-), BT79.2 (-), BT8.1 (+), BT80.1 (+), BT91.2 (-), BT92.1 (+), J1.6 (Pin_6), J3.8 (Pin_8)
- new net: BT102.2 (-), BT103.1 (+), BT114.2 (-), BT115.1 (+), BT18.2 (-), BT19.1 (+), BT30.2 (-), BT31.1 (+), BT42.2 (-), BT43.1 (+), BT54.2 (-), BT55.1 (+), BT6.2 (-), BT66.2 (-), BT67.1 (+), BT7.1 (+), BT78.2 (-), BT79.1 (+), BT90.2 (-), BT91.1 (+), J1.7 (Pin_7), J3.7 (Pin_7)
- new net: BT101.2 (-), BT102.1 (+), BT113.2 (-), BT114.1 (+), BT17.2 (-), BT18.1 (+), BT29.2 (-), BT30.1 (+), BT41.2 (-), BT42.1 (+), BT5.2 (-), BT53.2 (-), BT54.1 (+), BT6.1 (+), BT65.2 (-), BT66.1 (+), BT77.2 (-), BT78.1 (+), BT89.2 (-), BT90.1 (+), J1.8 (Pin_8), J3.6 (Pin_6)
- new net: BT100.2 (-), BT101.1 (+), BT112.2 (-), BT113.1 (+), BT16.2 (-), BT17.1 (+), BT28.2 (-), BT29.1 (+), BT4.2 (-), BT40.2 (-), BT41.1 (+), BT5.1 (+), BT52.2 (-), BT53.1 (+), BT64.2 (-), BT65.1 (+), BT76.2 (-), BT77.1 (+), BT88.2 (-), BT89.1 (+), J1.9 (Pin_9), J3.5 (Pin_5)
Other:
- moved on the sheet: BT10, BT106, BT107, BT108, BT11, BT118, BT119, BT12, BT120, BT22, BT23, BT24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

Commit message: small changes to top pcb
Parts:
- removed J2: Conn_01x10, Pin_Headers:Pin_Header_Straight_1x10_Pitch2.54mm, symbol Connector_Generic:Conn_01x10
- added C? (x10): 1u, symbol Device:C
- added C? (x2): 100n, symbol Device:C
- added J2, J?: Conn_01x04_Female, symbol Connector:Conn_01x04_Female
- added R? (x9): 100k, symbol Device:R
- added R?: 240, symbol Device:R
- added TH? (x3): Thermistor, Resistors_SMD:R_0805_HandSoldering, symbol Device:Thermistor
- added U?: ADC128D818, Package_SO:TSSOP-16_4.4x5mm_P0.65mm, symbol Analog_ADC:ADC128D818
Connections:
- net at TH3.1: now also U?.14 (IN2)
- net at TH3.2: now also C?.1, R?.2
- net at TH4.1: now also U?.13 (IN3)
- net at TH4.2: now also C?.1, R?.2
- net at TH5.1: now also U?.12 (IN4)
- net at TH5.2: now also C?.1, R?.2
- net at TH1.1: now also U?.16 (IN0)
- net at TH1.2: now also C?.1, R?.2
- net at TH2.1: now also U?.15 (IN1)
- net at TH2.2: now also C?.1, R?.2
- new net: C?.1, C?.1, R?.2, U?.1 (VREF)
- new net: TH?.1, U?.10 (IN6)
- new net: TH?.1, U?.11 (IN5)
- new net: J2.2 (Pin_2), J?.2 (Pin_2), U?.2 (SDA)
- new net: J2.3 (Pin_3), J?.3 (Pin_3), U?.3 (SCL)
- new net: R?.2, U?.6 (~INT)
- new net: TH?.1, U?.9 (IN7)
- new net: C?.1, R?.2, TH?.2 (x3)
- new net +5V: C?.1, C?.1, J2.1 (Pin_1), J?.1 (Pin_1), R?.1, R?.1, R?.1, R?.1, R?.1, R?.1, R?.1, R?.1, R?.1, R?.1, U?.5 (V+)
- new net GND: C?.2, C?.2, C?.2, C?.2, C?.2, C?.2, C?.2, C?.2, C?.2, C?.2, C?.2, C?.2, J2.4 (Pin_4), J?.4 (Pin_4), U?.4 (GND), U?.7 (A0), U?.8 (A1)
Other:
- moved on the sheet: TH1, TH2, TH3, TH4, TH5
