File: PCB/Pack/Pack.sch (KiCad schematic (older format))
At the start: 158 parts, among them J1 Conn_01x13, J14 Conn_01x01, J15 Conn_01x01, J2 Conn_01x04_Female, J3 Conn_01x13

Commit message: Minor changes
Parts:
- removed C? (x8): 1u, symbol Device:C
- removed C?: 100n, symbol Device:C
- removed J2, J?: Conn_01x04_Female, symbol Connector:Conn_01x04_Female
- removed R? (x7): 100k, symbol Device:R
- added C11: 100n, Capacitors_SMD:C_0603_HandSoldering, symbol Device:C
- added C12, C2, C3, C4, C5, C6, C7, C8: 1u, Capacitors_SMD:C_0603_HandSoldering, symbol Device:C
- added J2: Conn_01x04, Connectors_Molex:Molex_KK-6410-04_04x2.54mm_Straight, symbol Connector_Generic:Conn_01x04
- added J4: Conn_01x04, Pin_Headers:Pin_Header_Straight_1x04_Pitch2.54mm, symbol Connector_Generic:Conn_01x04
- added R2, R3, R4, R5, R6, R7, R8: 100k, Resistors_SMD:R_0603_HandSoldering, symbol Device:R
- C1, C10, C9: renamed from C?; footprint (none) -> Capacitors_SMD:C_0603_HandSoldering
- J3: footprint Pin_Headers:Pin_Header_Straight_1x13_Pitch2.54mm -> Connectors_Molex:Molex_KK-6410-13_13x2.54mm_Straight
- R1, R10, R9: renamed from R?; footprint (none) -> Resistors_SMD:R_0603_HandSoldering
- U1: renamed from U?; footprint Package_SO:TSSOP-16_4.4x5mm_P0.65mm -> Housings_SSOP:TSSOP-16_4.4x5mm_Pitch0.65mm
- gave numbers to parts that had none: 3
Connections:
- net +5V: now also C10.1, C9.1, J2.1 (Pin_1), J4.1 (Pin_1), R2.1, R3.1, R4.1, R5.1, R6.1, R7.1, R8.1
- net GND: now also C11.2, C12.2, C2.2, C3.2, C4.2, C5.2, C6.2, C7.2, C8.2, J2.4 (Pin_4), J4.4 (Pin_4)
- net at TH3.2: now also C6.1, R6.2
- net at TH4.2: now also C5.1, R5.2
- net at TH5.2: now also C4.1, R4.2
- net at R9.2, U1.1 (VREF): now also C11.1, C12.1; no longer C10.1, C9.1
- net at U1.2 (SDA): now also J2.2 (Pin_2), J4.2 (Pin_2)
- net at U1.3 (SCL): now also J2.3 (Pin_3), J4.3 (Pin_3)
- net at TH6.2: now also C3.1, R3.2
- net at TH1.2: now also C8.1, R8.2
- net at TH2.2: now also C7.1, R7.2
- net at TH7.2: now also C2.1, R2.2
Other:
- moved on the sheet: C10, C9

Commit message: Updated design
Other:
- moved on the sheet: BT1, BT10, BT100, BT101, BT102, BT103, BT104, BT105, BT106, BT107, BT108, BT109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
