File: PCB/Pack/pack.kicad_pcb (KiCad board)
At the start: 2 copper layers, 100 x 100 mm, 0 parts

Commit message: pack schematic & pcb
Parts:
- added BT1: Battery_Cell, ENNOID:Battery, F.Cu at (10.0, 24.2)
- added BT10: Battery_Cell, ENNOID:Battery, F.Cu at (40.0, 9.18)
- added BT11: Battery_Cell, ENNOID:Battery, F.Cu at (40.0, 42.5)
- added BT12: Battery_Cell, ENNOID:Battery, F.Cu at (40.0, 75.8)
- added BT13: Battery_Cell, ENNOID:Battery, F.Cu at (50.0, 24.2)
- added BT14: Battery_Cell, ENNOID:Battery, F.Cu at (50.0, 57.5)
- added BT15: Battery_Cell, ENNOID:Battery, F.Cu at (50.0, 90.8)
- added BT16: Battery_Cell, ENNOID:Battery, F.Cu at (60.0, 9.18)
- added BT17: Battery_Cell, ENNOID:Battery, F.Cu at (60.0, 42.5)
- added BT18: Battery_Cell, ENNOID:Battery, F.Cu at (60.0, 75.8)
- added BT19: Battery_Cell, ENNOID:Battery, F.Cu at (70.0, 24.2)
- added BT2: Battery_Cell, ENNOID:Battery, F.Cu at (10.0, 57.5)
- added BT20: Battery_Cell, ENNOID:Battery, F.Cu at (70.0, 57.5)
- added BT21: Battery_Cell, ENNOID:Battery, F.Cu at (70.0, 90.8)
- added BT22: Battery_Cell, ENNOID:Battery, F.Cu at (80.0, 9.18)
- added BT23: Battery_Cell, ENNOID:Battery, F.Cu at (80.0, 42.5)
- added BT24: Battery_Cell, ENNOID:Battery, F.Cu at (80.0, 75.8)
- added BT25: Battery_Cell, ENNOID:Battery, F.Cu at (90.0, 24.2)
- added BT26: Battery_Cell, ENNOID:Battery, F.Cu at (90.0, 57.5)
- added BT27: Battery_Cell, ENNOID:Battery, F.Cu at (90.0, 90.8)
- added BT28: Battery_Cell, ENNOID:Battery, F.Cu at (100.0, 9.18)
- added BT29: Battery_Cell, ENNOID:Battery, F.Cu at (100.0, 42.5)
- added BT3: Battery_Cell, ENNOID:Battery, F.Cu at (10.0, 90.8)
- added BT30: Battery_Cell, ENNOID:Battery, F.Cu at (100.0, 75.8)
- added BT31: Battery_Cell, ENNOID:Battery, F.Cu at (0.00, 9.18)
- added BT32: Battery_Cell, ENNOID:Battery, F.Cu at (0.00, 42.5)
- added BT33: Battery_Cell, ENNOID:Battery, F.Cu at (0.00, 75.8)
- added BT4: Battery_Cell, ENNOID:Battery, F.Cu at (20.0, 9.18)
- added BT5: Battery_Cell, ENNOID:Battery, F.Cu at (20.0, 42.5)
- added BT6: Battery_Cell, ENNOID:Battery, F.Cu at (20.0, 75.8)
- added BT7: Battery_Cell, ENNOID:Battery, F.Cu at (30.0, 24.2)
- added BT8: Battery_Cell, ENNOID:Battery, F.Cu at (30.0, 57.5)
- added BT9: Battery_Cell, ENNOID:Battery, F.Cu at (30.0, 90.8)
Routing:
- net Net-(BT11-Pad2): track 0.00 -> 415.0 mm
- net Net-(BT1-Pad2): track 0.00 -> 412.5 mm
- net Net-(BT1-Pad1): track 0.00 -> 167.5 mm
- net Net-(BT12-Pad2): track 0.00 -> 119.6 mm
Other:
- outline, holes or cut-outs redrawn
- rule pad_to_mask_clearance: 0.2 -> 0.051

Commit message: pack update
Parts:
- added F1: Fuse, Resistors_SMD:R_0805, F.Cu at (5.00, 5.00)
- added F10: Fuse, Resistors_SMD:R_0805, F.Cu at (35.0, 14.0)
- added F11: Fuse, Resistors_SMD:R_0805, F.Cu at (35.0, 47.0)
- added F12: Fuse, Resistors_SMD:R_0805, F.Cu at (35.0, 80.0)
- added F13: Fuse, Resistors_SMD:R_0805, F.Cu at (45.0, 5.00)
- added F14: Fuse, Resistors_SMD:R_0805, F.Cu at (40.0, 35.0)
- added F15: Fuse, Resistors_SMD:R_0805, F.Cu at (40.0, 68.0)
- added F16: Fuse, Resistors_SMD:R_0805, F.Cu at (55.0, 14.0)
- added F17: Fuse, Resistors_SMD:R_0805, F.Cu at (55.0, 47.0)
- added F18: Fuse, Resistors_SMD:R_0805, F.Cu at (55.0, 80.0)
- added F19: Fuse, Resistors_SMD:R_0805, F.Cu at (65.0, 5.00)
- added F2: Fuse, Resistors_SMD:R_0805, F.Cu at (1.00, 35.0)
- added F20: Fuse, Resistors_SMD:R_0805, F.Cu at (60.0, 35.0)
- added F21: Fuse, Resistors_SMD:R_0805, F.Cu at (60.0, 68.0)
- added F22: Fuse, Resistors_SMD:R_0805, F.Cu at (75.0, 14.0)
- added F23: Fuse, Resistors_SMD:R_0805, F.Cu at (75.0, 47.0)
- added F24: Fuse, Resistors_SMD:R_0805, F.Cu at (75.0, 80.0)
- added F25: Fuse, Resistors_SMD:R_0805, F.Cu at (85.0, 5.00)
- added F26: Fuse, Resistors_SMD:R_0805, F.Cu at (80.0, 35.0)
- added F27: Fuse, Resistors_SMD:R_0805, F.Cu at (80.0, 68.0)
- added F28: Fuse, Resistors_SMD:R_0805, F.Cu at (95.0, 14.0)
- added F29: Fuse, Resistors_SMD:R_0805, F.Cu at (95.0, 47.0)
- added F3: Fuse, Resistors_SMD:R_0805, F.Cu at (1.00, 68.0)
- added F30: Fuse, Resistors_SMD:R_0805, F.Cu at (95.0, 80.0)
- added F31: Fuse, Resistors_SMD:R_0805, F.Cu at (95.0, 5.00)
- added F32: Fuse, Resistors_SMD:R_0805, F.Cu at (98.0, 35.0)
- added F33: Fuse, Resistors_SMD:R_0805, F.Cu at (98.0, 68.0)
- added F4: Fuse, Resistors_SMD:R_0805, F.Cu at (15.0, 14.0)
- added F5: Fuse, Resistors_SMD:R_0805, F.Cu at (15.0, 47.0)
- added F6: Fuse, Resistors_SMD:R_0805, F.Cu at (15.0, 80.0)
- added F7: Fuse, Resistors_SMD:R_0805, F.Cu at (25.0, 5.00)
- added F8: Fuse, Resistors_SMD:R_0805, F.Cu at (20.0, 35.0)
- added F9: Fuse, Resistors_SMD:R_0805, F.Cu at (20.0, 68.0)
- added J1: Conn_01x01, Pin_Headers:Pin_Header_Straight_1x01_Pitch2.54mm, F.Cu at (-26.0, 8.00)
- added J2: Conn_01x01, Pin_Headers:Pin_Header_Straight_1x01_Pitch2.54mm, F.Cu at (-17.0, 33.0)
- added J3: Conn_01x01, Pin_Headers:Pin_Header_Straight_1x01_Pitch2.54mm, F.Cu at (-29.0, 66.0)
- added J4: Conn_01x01, Pin_Headers:Pin_Header_Straight_1x01_Pitch2.54mm, F.Cu at (-35.0, 91.0)
- added J5: Conn_01x01, ENNOID:Pack, B.Cu at (50.0, 1.50)
- added J6: Conn_01x01, ENNOID:Pack, B.Cu at (50.0, 98.5)
- added J7: Conn_01x02, Pin_Headers:Pin_Header_Straight_1x02_Pitch2.54mm, F.Cu at (89.0, 73.0)
- added J8: Conn_01x02, Pin_Headers:Pin_Header_Straight_1x02_Pitch2.54mm, F.Cu at (89.0, 39.0)
- added J9: Conn_01x02, Pin_Headers:Pin_Header_Straight_1x02_Pitch2.54mm, F.Cu at (88.0, -6.00)
- added TH1: Thermistor, Resistors_THT:R_Axial_DIN0309_L9.0mm_D3.2mm_P5.08mm_Vertical, F.Cu at (88.0, 69.0)
- added TH2: Thermistor, Resistors_THT:R_Axial_DIN0309_L9.0mm_D3.2mm_P5.08mm_Vertical, F.Cu at (78.0, -4.00)
- added TH3: Thermistor, Resistors_THT:R_Axial_DIN0309_L9.0mm_D3.2mm_P5.08mm_Vertical, F.Cu at (88.0, 35.0)
Connections:
- BT10 pad 1: Net-(BT1-Pad1) -> Net-(BT10-Pad1)
- BT11 pad 1: Net-(BT1-Pad2) -> Net-(BT11-Pad1)
- BT12 pad 1: Net-(BT11-Pad2) -> Net-(BT12-Pad1)
- BT13 pad 1: Net-(BT1-Pad1) -> Net-(BT13-Pad1)
- BT14 pad 1: Net-(BT1-Pad2) -> Net-(BT14-Pad1)
- BT15 pad 1: Net-(BT11-Pad2) -> Net-(BT15-Pad1)
- BT16 pad 1: Net-(BT1-Pad1) -> Net-(BT16-Pad1)
- BT17 pad 1: Net-(BT1-Pad2) -> Net-(BT17-Pad1)
- BT18 pad 1: Net-(BT11-Pad2) -> Net-(BT18-Pad1)
- BT19 pad 1: Net-(BT1-Pad1) -> Net-(BT19-Pad1)
- BT2 pad 1: Net-(BT1-Pad2) -> Net-(BT2-Pad1)
- BT20 pad 1: Net-(BT1-Pad2) -> Net-(BT20-Pad1)
- BT21 pad 1: Net-(BT11-Pad2) -> Net-(BT21-Pad1)
- BT22 pad 1: Net-(BT1-Pad1) -> Net-(BT22-Pad1)
- BT23 pad 1: Net-(BT1-Pad2) -> Net-(BT23-Pad1)
- BT24 pad 1: Net-(BT11-Pad2) -> Net-(BT24-Pad1)
- BT25 pad 1: Net-(BT1-Pad1) -> Net-(BT25-Pad1)
- BT26 pad 1: Net-(BT1-Pad2) -> Net-(BT26-Pad1)
- BT27 pad 1: Net-(BT11-Pad2) -> Net-(BT27-Pad1)
- BT28 pad 1: Net-(BT1-Pad1) -> Net-(BT28-Pad1)
- BT29 pad 1: Net-(BT1-Pad2) -> Net-(BT29-Pad1)
- BT3 pad 1: Net-(BT11-Pad2) -> Net-(BT3-Pad1)
- BT30 pad 1: Net-(BT11-Pad2) -> Net-(BT30-Pad1)
- BT31 pad 1: Net-(BT1-Pad1) -> Net-(BT31-Pad1)
- BT32 pad 1: Net-(BT1-Pad2) -> Net-(BT32-Pad1)
- BT33 pad 1: Net-(BT11-Pad2) -> Net-(BT33-Pad1)
- BT4 pad 1: Net-(BT1-Pad1) -> Net-(BT4-Pad1)
- BT5 pad 1: Net-(BT1-Pad2) -> Net-(BT5-Pad1)
- BT6 pad 1: Net-(BT11-Pad2) -> Net-(BT6-Pad1)
- BT7 pad 1: Net-(BT1-Pad1) -> Net-(BT7-Pad1)
- BT8 pad 1: Net-(BT1-Pad2) -> Net-(BT8-Pad1)
- BT9 pad 1: Net-(BT11-Pad2) -> Net-(BT9-Pad1)
Routing:
- net Net-(BT11-Pad2): track 415.0 -> 0.00 mm
- net Net-(BT1-Pad2): track 412.5 -> 0.00 mm
- net Net-(BT1-Pad1): track 167.5 -> 0.00 mm
- net Net-(BT12-Pad2): track 119.6 -> 0.00 mm
- net Net-(BT6-Pad1): track 0.00 -> 6.90 mm
- net Net-(J8-Pad2): track 0.00 -> 4.64 mm
- net Net-(J7-Pad2): track 0.00 -> 4.64 mm
- net Net-(J8-Pad1): track 0.00 -> 4.41 mm
- net Net-(J7-Pad1): track 0.00 -> 4.41 mm
- added copper zone on B.Cu, net Net-(BT1-Pad1)
- added copper zone on B.Cu, net Net-(BT12-Pad2)

Commit message: Pack completed
Parts:
- removed J9: Conn_01x02, Pin_Headers:Pin_Header_Straight_1x02_Pitch2.54mm
- removed TH2: Thermistor, Resistors_THT:R_Axial_DIN0309_L9.0mm_D3.2mm_P5.08mm_Vertical
- F1, F10, F11, F12, F13, F14, F15, F16, F17, F18, F19, F2, F20, F21, F22, F23, F24, F25, F26, F27, F28, F29, F3, F30, F31, F32, F33, F4, F5, F6, F7, F8, F9: footprint Resistors_SMD:R_0805 -> Fuse_Holders_and_Fuses:Fuse_SMD1206_Wave; moved to B.Cu
- J1, J2, J3, J4: moved to B.Cu
- moved J4 55.0 mm to (20.0, 92.5)
- moved J3 39.2 mm to (10.0, 70.0)
- moved J1 36.0 mm to (10.0, 8.00)
- moved J2 27.1 mm to (10.0, 35.0)
- moved J7 18.4 mm to (71.0, 69.0), turned to 270 degrees
- moved J8 18.4 mm to (71.0, 35.0), turned to 270 degrees
- moved F10 10.0 mm to (25.0, 14.0)
- moved F11 10.0 mm to (25.0, 47.0)
- moved F16 10.0 mm to (45.0, 14.0)
- moved F17 10.0 mm to (45.0, 47.0)
- moved F22 10.0 mm to (65.0, 14.0)
- moved F23 10.0 mm to (65.0, 47.0)
- moved F28 10.0 mm to (85.0, 14.0)
- moved F29 10.0 mm to (85.0, 47.0)
- moved F4 10.0 mm to (5.00, 14.0)
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Routing:
- net Net-(BT1-Pad2): track 0.00 -> 281.5 mm
- net Net-(BT11-Pad2): track 0.00 -> 280.4 mm
- net Net-(BT12-Pad2): track 0.00 -> 120.9 mm
- net Net-(F1-Pad1): track 0.00 -> 42.4 mm
- net Net-(J8-Pad2): track 4.64 -> 27.1 mm
- net Net-(J7-Pad2): track 4.64 -> 26.3 mm
- net Net-(J8-Pad1): track 4.41 -> 17.0 mm
- net Net-(J7-Pad1): track 4.41 -> 17.0 mm
- net Net-(BT9-Pad1): track 0.00 -> 11.3 mm
- net Net-(BT3-Pad1): track 0.00 -> 11.3 mm
- net Net-(BT27-Pad1): track 0.00 -> 11.3 mm
- net Net-(BT21-Pad1): track 0.00 -> 11.3 mm
- net Net-(BT15-Pad1): track 0.00 -> 11.3 mm
- net Net-(BT8-Pad1): track 0.00 -> 11.0 mm
- net Net-(BT26-Pad1): track 0.00 -> 11.0 mm
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- added copper zone on B.Cu, net Net-(F1-Pad1)
- removed copper zone on B.Cu, net Net-(BT1-Pad1)
