File: PCB/Pack/pack.kicad_pcb (KiCad board)
At the start: 2 copper layers, 100 x 100 mm, 43 parts, among them J1 Conn_01x01, J2 Conn_01x01, J3 Conn_01x01, J4 Conn_01x01, J5 Conn_01x01, J6 Conn_01x01, J7 Conn_01x02, J8 Conn_01x02

Commit message: Traces
Parts:
- moved J7 44.7 mm to (114.5, 55.5)
- moved J8 43.4 mm to (114.5, 28.5)
- moved TH3 36.2 mm to (124.0, 28.5)
- moved J2 27.1 mm to (-17.0, 30.0)
- moved TH1 26.2 mm to (113.5, 61.0)
- moved J3 25.0 mm to (-15.0, 65.5)
Routing:
- net Net-(BT12-Pad2): vias 0 -> 294
- net Net-(BT11-Pad2): vias 0 -> 195
- net Net-(BT1-Pad2): vias 0 -> 195
- added copper zone on B.Cu, net Net-(BT1-Pad2)
- added copper zone on F.Cu, net Net-(BT1-Pad2)
- added copper zone on B.Cu, net Net-(BT11-Pad2)
- added copper zone on F.Cu, net Net-(BT11-Pad2)
- added copper zone on F.Cu, net Net-(BT12-Pad2)

Commit message: PCB major changes
Parts:
- added J9: Conn_01x02, Pin_Headers:Pin_Header_Straight_1x02_Pitch2.54mm_SMD_Pin1Left, B.Cu at (50.4, 5.80)
- added TH2: Thermistor, Resistors_SMD:R_0805_HandSoldering, B.Cu at (50.0, 9.90)
- BT31, BT32, BT33: footprint ENNOID:Battery -> ENNOID:18650
- J7, J8: footprint Pin_Headers:Pin_Header_Straight_1x02_Pitch2.54mm -> Pin_Headers:Pin_Header_Straight_1x02_Pitch2.54mm_SMD_Pin1Left; moved to B.Cu
- TH1, TH3: footprint Resistors_THT:R_Axial_DIN0309_L9.0mm_D3.2mm_P5.08mm_Vertical -> Resistors_SMD:R_0805_HandSoldering; moved to B.Cu
- moved TH3 75.4 mm to (50.0, 43.2)
- moved J2 67.1 mm to (50.0, 33.3)
- moved J7 66.2 mm to (50.5, 72.5), turned to 0 degrees
- moved TH1 65.4 mm to (50.0, 76.6)
- moved J3 65.0 mm to (50.0, 66.6)
- moved J8 64.9 mm to (50.5, 39.1), turned to 0 degrees
- moved J1 37.1 mm to (50.0, 1.30)
- moved J4 26.4 mm to (50.0, 98.7), turned to 180 degrees
- moved J5 0.50 mm to (50.0, 1.25)
- moved J6 0.50 mm to (50.0, 98.8)
Routing:
- net Net-(J8-Pad2): track 0.00 -> 5.70 mm
- net Net-(J7-Pad2): track 0.00 -> 5.70 mm
- net Net-(J9-Pad2): track 0.00 -> 5.66 mm
- net Net-(J8-Pad1): track 0.00 -> 3.47 mm
- net Net-(J7-Pad1): track 0.00 -> 2.91 mm
- net Net-(J9-Pad1): track 0.00 -> 2.87 mm
- net Net-(BT11-Pad2): vias 195 -> 198
- net Net-(BT1-Pad2): vias 195 -> 198
Other:
- board text added: "C3 C6 C9 C12 C15"

Commit message: Final version
Parts:
- BT1, BT10, BT11, BT12, BT13, BT14, BT15, BT16, BT17, BT18, BT19, BT2, BT20, BT21, BT22, BT23, BT24, BT25, BT26, BT27, BT3, BT4, BT5, BT6, BT7, BT8, BT9: moved to B.Cu
- BT28, BT29, BT30, BT31, BT32, BT33: footprint ENNOID:18650 -> ENNOID:half; moved to B.Cu
- moved J9 0.30 mm to (50.1, 5.80)
- turned BT1 to 0 degrees
- turned BT10 to 180 degrees
- turned BT11 to 180 degrees
- turned BT12 to 180 degrees
- turned BT13 to 0 degrees
- turned BT14 to 0 degrees
- turned BT15 to 0 degrees
- turned BT16 to 180 degrees
- turned BT17 to 180 degrees
- turned BT18 to 180 degrees
- turned BT19 to 0 degrees
- turned BT2 to 0 degrees
- turned BT20 to 0 degrees
- turned BT21 to 0 degrees
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Routing:
- net Net-(BT11-Pad2): vias 198 -> 200
- net Net-(BT1-Pad2): vias 198 -> 200
Other:
- outline, holes or cut-outs redrawn
- board text added: "C12"
- board text added: "C18"
- board text removed: "C3 C6 C9 C12 C15"

Commit message: Major update 12S10P
3dprintable casing for 12S10P 1.5kWh
Parts:
- removed J4: Conn_01x01, Pin_Headers:Pin_Header_Straight_1x01_Pitch2.54mm
- removed J5, J6: Conn_01x01, ENNOID:Pack
- removed J7, J8, J9: Conn_01x02, Pin_Headers:Pin_Header_Straight_1x02_Pitch2.54mm_SMD_Pin1Left
- added BT1: Battery_Cell, ENNOID:18650, F.Cu at (240.0, 9.12)
- added BT100: Battery_Cell, ENNOID:18650, F.Cu at (180.0, 147.7)
- added BT101: Battery_Cell, ENNOID:18650, F.Cu at (160.0, 147.7)
- added BT102: Battery_Cell, ENNOID:18650, F.Cu at (140.0, 147.7)
- added BT103: Battery_Cell, ENNOID:18650, F.Cu at (120.0, 147.7)
- added BT104: Battery_Cell, ENNOID:18650, F.Cu at (100.0, 147.7)
- added BT105: Battery_Cell, ENNOID:18650, F.Cu at (80.0, 147.7)
- added BT109: Battery_Cell, ENNOID:18650, F.Cu at (230.0, 165.0)
- added BT110: Battery_Cell, ENNOID:18650, F.Cu at (210.0, 165.0)
- added BT111: Battery_Cell, ENNOID:18650, F.Cu at (190.0, 165.0)
- added BT112: Battery_Cell, ENNOID:18650, F.Cu at (170.0, 165.0)
- added BT113: Battery_Cell, ENNOID:18650, F.Cu at (150.0, 165.0)
- added BT114: Battery_Cell, ENNOID:18650, F.Cu at (130.0, 165.0)
- added BT115: Battery_Cell, ENNOID:18650, F.Cu at (110.0, 165.0)
- added BT116: Battery_Cell, ENNOID:18650, F.Cu at (90.0, 165.0)
- added BT117: Battery_Cell, ENNOID:18650, F.Cu at (70.0, 165.0)
- added BT118: Battery_Cell, ENNOID:18650, F.Cu at (50.0, 165.0)
- added BT119: Battery_Cell, ENNOID:18650, F.Cu at (30.0, 165.0)
- added BT120: Battery_Cell, ENNOID:18650, F.Cu at (10.0, 165.0)
- added BT13: Battery_Cell, ENNOID:18650, F.Cu at (230.0, 26.4)
- added BT14: Battery_Cell, ENNOID:18650, F.Cu at (210.0, 26.4)
- added BT15: Battery_Cell, ENNOID:18650, F.Cu at (190.0, 26.4)
- added BT16: Battery_Cell, ENNOID:18650, F.Cu at (170.0, 26.4)
- added BT17: Battery_Cell, ENNOID:18650, F.Cu at (150.0, 26.4)
- added BT18: Battery_Cell, ENNOID:18650, F.Cu at (130.0, 26.4)
- added BT19: Battery_Cell, ENNOID:18650, F.Cu at (110.0, 26.4)
- added BT2: Battery_Cell, ENNOID:18650, F.Cu at (220.0, 9.12)
- added BT20: Battery_Cell, ENNOID:18650, F.Cu at (90.0, 26.4)
- added BT21: Battery_Cell, ENNOID:18650, F.Cu at (70.0, 26.4)
- added BT25: Battery_Cell, ENNOID:18650, F.Cu at (240.0, 43.8)
- added BT26: Battery_Cell, ENNOID:18650, F.Cu at (220.0, 43.8)
- added BT27: Battery_Cell, ENNOID:18650, F.Cu at (200.0, 43.8)
- added BT3: Battery_Cell, ENNOID:18650, F.Cu at (200.0, 9.12)
- added BT37: Battery_Cell, ENNOID:18650, F.Cu at (230.0, 61.1)
- added BT38: Battery_Cell, ENNOID:18650, F.Cu at (210.0, 61.1)
- added BT39: Battery_Cell, ENNOID:18650, F.Cu at (190.0, 61.1)
- added BT4: Battery_Cell, ENNOID:18650, F.Cu at (180.0, 9.12)
- added BT40: Battery_Cell, ENNOID:18650, F.Cu at (170.0, 61.1)
- added BT41: Battery_Cell, ENNOID:18650, F.Cu at (150.0, 61.1)
- added BT42: Battery_Cell, ENNOID:18650, F.Cu at (130.0, 61.1)
- added BT43: Battery_Cell, ENNOID:18650, F.Cu at (110.0, 61.1)
- added BT44: Battery_Cell, ENNOID:18650, F.Cu at (90.0, 61.1)
- added BT45: Battery_Cell, ENNOID:18650, F.Cu at (70.0, 61.1)
- added BT49: Battery_Cell, ENNOID:18650, F.Cu at (240.0, 78.4)
- added BT5: Battery_Cell, ENNOID:18650, F.Cu at (160.0, 9.12)
- added BT50: Battery_Cell, ENNOID:18650, F.Cu at (220.0, 78.4)
- added BT51: Battery_Cell, ENNOID:18650, F.Cu at (200.0, 78.4)
- added BT52: Battery_Cell, ENNOID:18650, F.Cu at (180.0, 78.4)
- added BT53: Battery_Cell, ENNOID:18650, F.Cu at (160.0, 78.4)
- added BT54: Battery_Cell, ENNOID:18650, F.Cu at (140.0, 78.4)
- added BT55: Battery_Cell, ENNOID:18650, F.Cu at (120.0, 78.4)
- added BT56: Battery_Cell, ENNOID:18650, F.Cu at (100.0, 78.4)
- added BT57: Battery_Cell, ENNOID:18650, F.Cu at (80.0, 78.4)
- added BT6: Battery_Cell, ENNOID:18650, F.Cu at (140.0, 9.12)
- added BT61: Battery_Cell, ENNOID:18650, F.Cu at (230.0, 95.7)
- added BT62: Battery_Cell, ENNOID:18650, F.Cu at (210.0, 95.7)
- added BT63: Battery_Cell, ENNOID:18650, F.Cu at (190.0, 95.7)
- added BT64: Battery_Cell, ENNOID:18650, F.Cu at (170.0, 95.7)
- added BT65: Battery_Cell, ENNOID:18650, F.Cu at (150.0, 95.7)
- added BT66: Battery_Cell, ENNOID:18650, F.Cu at (130.0, 95.7)
- added BT67: Battery_Cell, ENNOID:18650, F.Cu at (110.0, 95.7)
- added BT68: Battery_Cell, ENNOID:18650, F.Cu at (90.0, 95.7)
- added BT69: Battery_Cell, ENNOID:18650, F.Cu at (70.0, 95.7)
- added BT7: Battery_Cell, ENNOID:18650, F.Cu at (120.0, 9.12)
- added BT73: Battery_Cell, ENNOID:18650, F.Cu at (240.0, 113.0)
- added BT74: Battery_Cell, ENNOID:18650, F.Cu at (220.0, 113.0)
- added BT75: Battery_Cell, ENNOID:18650, F.Cu at (200.0, 113.0)
- added BT76: Battery_Cell, ENNOID:18650, F.Cu at (180.0, 113.0)
- added BT77: Battery_Cell, ENNOID:18650, F.Cu at (160.0, 113.0)
- added BT78: Battery_Cell, ENNOID:18650, F.Cu at (140.0, 113.0)
- added BT79: Battery_Cell, ENNOID:18650, F.Cu at (120.0, 113.0)
- added BT8: Battery_Cell, ENNOID:18650, F.Cu at (100.0, 9.12)
- added BT80: Battery_Cell, ENNOID:18650, F.Cu at (100.0, 113.0)
- added BT81: Battery_Cell, ENNOID:18650, F.Cu at (80.0, 113.0)
- added BT85: Battery_Cell, ENNOID:18650, F.Cu at (230.0, 130.4)
- added BT86: Battery_Cell, ENNOID:18650, F.Cu at (210.0, 130.4)
- added BT87: Battery_Cell, ENNOID:18650, F.Cu at (190.0, 130.4)
- added BT88: Battery_Cell, ENNOID:18650, F.Cu at (170.0, 130.4)
- added BT89: Battery_Cell, ENNOID:18650, F.Cu at (150.0, 130.4)
- added BT9: Battery_Cell, ENNOID:18650, F.Cu at (80.0, 9.12)
- added BT90: Battery_Cell, ENNOID:18650, F.Cu at (130.0, 130.4)
- added BT91: Battery_Cell, ENNOID:18650, F.Cu at (110.0, 130.4)
- added BT92: Battery_Cell, ENNOID:18650, F.Cu at (90.0, 130.4)
- added BT93: Battery_Cell, ENNOID:18650, F.Cu at (70.0, 130.4)
- added BT97: Battery_Cell, ENNOID:18650, F.Cu at (240.0, 147.7)
- added BT98: Battery_Cell, ENNOID:18650, F.Cu at (220.0, 147.7)
- added BT99: Battery_Cell, ENNOID:18650, F.Cu at (200.0, 147.7)
- added J14: Conn_01x01, ENNOID:Pack, F.Cu at (250.0, 87.0)
- added J15: Conn_01x01, ENNOID:Pack, F.Cu at (0.00, 87.0)
- added LOGO1: Logo_Open_Hardware_Small, ENNOID:ENNOID-LOGO, B.Cu at (126.9, 87.2)
- added TH4: Thermistor, Resistors_SMD:R_0805_HandSoldering, F.Cu at (167.5, 70.4)
- added TH5: Thermistor, Resistors_SMD:R_0805_HandSoldering, F.Cu at (207.4, 35.0)
- BT10: renamed from BT1; moved to F.Cu
- BT106: renamed from BT25; moved to F.Cu
- BT107: renamed from BT26; moved to F.Cu
- BT108: renamed from BT27; moved to F.Cu
- BT11: renamed from BT2; moved to F.Cu
- BT12: renamed from BT3; moved to F.Cu
- BT22: renamed from BT4; moved to F.Cu
- BT23: renamed from BT5; moved to F.Cu
- BT24: renamed from BT6; moved to F.Cu
- BT28, BT29, BT30, BT31, BT32, BT33: footprint ENNOID:half -> ENNOID:18650; moved to F.Cu
- BT34: renamed from BT7; moved to F.Cu
- BT35: renamed from BT8; moved to F.Cu
- BT36: renamed from BT9; moved to F.Cu
- BT46: renamed from BT10; moved to F.Cu
- BT47: renamed from BT11; moved to F.Cu
- BT48: renamed from BT12; moved to F.Cu
- BT58: renamed from BT13; moved to F.Cu
- BT59: renamed from BT14; moved to F.Cu
- BT60: renamed from BT15; moved to F.Cu
- BT70: renamed from BT16; moved to F.Cu
- BT71: renamed from BT17; moved to F.Cu
- BT72: renamed from BT18; moved to F.Cu
- BT82: renamed from BT19; moved to F.Cu
- BT83: renamed from BT20; moved to F.Cu
- BT84: renamed from BT21; moved to F.Cu
- BT94: renamed from BT22; moved to F.Cu
- BT95: renamed from BT23; moved to F.Cu
- BT96: renamed from BT24; moved to F.Cu
- J1, J3: value Conn_01x01 -> Conn_01x13; footprint Pin_Headers:Pin_Header_Straight_1x01_Pitch2.54mm -> Pin_Headers:Pin_Header_Straight_1x13_Pitch2.54mm; moved to F.Cu
- J2: value Conn_01x01 -> Conn_01x10; footprint Pin_Headers:Pin_Header_Straight_1x01_Pitch2.54mm -> Pin_Headers:Pin_Header_Straight_1x10_Pitch2.54mm; moved to F.Cu
- TH1, TH2, TH3: moved to F.Cu
- moved J1 202.0 mm to (127.0, 188.0), turned to 90 degrees
- moved J2 162.0 mm to (98.0, 188.0), turned to 90 degrees
- moved J3 128.6 mm to (157.5, -4.00), turned to 270 degrees
- moved BT106 127.1 mm to (60.0, 147.7), turned to 270 degrees
- moved BT31 124.9 mm to (120.0, 43.8), turned to 270 degrees
- moved BT94 124.8 mm to (50.0, 130.4), turned to 270 degrees
- moved BT107 103.1 mm to (40.0, 147.7), turned to 270 degrees
- moved BT95 101.1 mm to (30.0, 130.4), turned to 270 degrees
- moved BT32 100.0 mm to (100.0, 43.8), turned to 270 degrees
- moved TH2 96.9 mm to (66.6, 105.4)
- moved BT108 90.2 mm to (20.0, 147.7), turned to 270 degrees
- moved BT82 89.5 mm to (60.0, 113.0), turned to 270 degrees
- moved BT96 88.7 mm to (10.0, 130.4)
- moved BT28 87.2 mm to (180.0, 43.8), turned to 270 degrees
- moved BT70 87.1 mm to (50.0, 95.7), turned to 270 degrees
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Connections:
- BT10 pad 1: Net-(BT1-Pad1) -> Net-(BT10-Pad1)
- BT10 pad 2: Net-(BT1-Pad2) -> Net-(BT10-Pad2)
- BT106 pad 1: Net-(BT1-Pad1) -> Net-(BT10-Pad1)
- BT106 pad 2: Net-(BT1-Pad2) -> Net-(BT10-Pad2)
- BT107 pad 1: Net-(BT1-Pad2) -> Net-(BT10-Pad2)
- BT107 pad 2: Net-(BT11-Pad2) -> Net-(BT107-Pad2)
- BT108 pad 1: Net-(BT11-Pad2) -> Net-(BT107-Pad2)
- BT108 pad 2: Net-(BT12-Pad2) -> Net-(BT108-Pad2)
- BT11 pad 1: Net-(BT1-Pad2) -> Net-(BT10-Pad2)
- BT11 pad 2: Net-(BT11-Pad2) -> Net-(BT107-Pad2)
- BT12 pad 1: Net-(BT11-Pad2) -> Net-(BT107-Pad2)
- BT12 pad 2: Net-(BT12-Pad2) -> Net-(BT108-Pad2)
- BT22 pad 1: Net-(BT1-Pad1) -> Net-(BT10-Pad1)
- BT22 pad 2: Net-(BT1-Pad2) -> Net-(BT10-Pad2)
- BT23 pad 1: Net-(BT1-Pad2) -> Net-(BT10-Pad2)
- BT23 pad 2: Net-(BT11-Pad2) -> Net-(BT107-Pad2)
- BT24 pad 1: Net-(BT11-Pad2) -> Net-(BT107-Pad2)
- BT24 pad 2: Net-(BT12-Pad2) -> Net-(BT108-Pad2)
- BT28 pad 1: Net-(BT1-Pad1) -> Net-(BT100-Pad1)
- BT28 pad 2: Net-(BT1-Pad2) -> Net-(BT100-Pad2)
- BT29 pad 1: Net-(BT1-Pad2) -> Net-(BT100-Pad2)
- BT29 pad 2: Net-(BT11-Pad2) -> Net-(BT101-Pad2)
- BT30 pad 1: Net-(BT11-Pad2) -> Net-(BT101-Pad2)
- BT30 pad 2: Net-(BT12-Pad2) -> Net-(BT102-Pad2)
- BT31 pad 1: Net-(BT1-Pad1) -> Net-(BT102-Pad2)
- BT31 pad 2: Net-(BT1-Pad2) -> Net-(BT103-Pad2)
- BT32 pad 1: Net-(BT1-Pad2) -> Net-(BT103-Pad2)
- BT32 pad 2: Net-(BT11-Pad2) -> Net-(BT104-Pad2)
- BT33 pad 1: Net-(BT11-Pad2) -> Net-(BT104-Pad2)
- BT33 pad 2: Net-(BT12-Pad2) -> Net-(BT10-Pad1)
- BT34 pad 1: Net-(BT1-Pad1) -> Net-(BT10-Pad1)
- BT34 pad 2: Net-(BT1-Pad2) -> Net-(BT10-Pad2)
- BT35 pad 1: Net-(BT1-Pad2) -> Net-(BT10-Pad2)
- BT35 pad 2: Net-(BT11-Pad2) -> Net-(BT107-Pad2)
- BT36 pad 1: Net-(BT11-Pad2) -> Net-(BT107-Pad2)
- BT36 pad 2: Net-(BT12-Pad2) -> Net-(BT108-Pad2)
- BT46 pad 1: Net-(BT1-Pad1) -> Net-(BT10-Pad1)
- BT46 pad 2: Net-(BT1-Pad2) -> Net-(BT10-Pad2)
- BT47 pad 1: Net-(BT1-Pad2) -> Net-(BT10-Pad2)
- BT47 pad 2: Net-(BT11-Pad2) -> Net-(BT107-Pad2)
- BT48 pad 1: Net-(BT11-Pad2) -> Net-(BT107-Pad2)
- BT48 pad 2: Net-(BT12-Pad2) -> Net-(BT108-Pad2)
- BT58 pad 1: Net-(BT1-Pad1) -> Net-(BT10-Pad1)
- BT58 pad 2: Net-(BT1-Pad2) -> Net-(BT10-Pad2)
- BT59 pad 1: Net-(BT1-Pad2) -> Net-(BT10-Pad2)
- BT59 pad 2: Net-(BT11-Pad2) -> Net-(BT107-Pad2)
- BT60 pad 1: Net-(BT11-Pad2) -> Net-(BT107-Pad2)
- BT60 pad 2: Net-(BT12-Pad2) -> Net-(BT108-Pad2)
- BT70 pad 1: Net-(BT1-Pad1) -> Net-(BT10-Pad1)
- BT70 pad 2: Net-(BT1-Pad2) -> Net-(BT10-Pad2)
- BT71 pad 1: Net-(BT1-Pad2) -> Net-(BT10-Pad2)
- BT71 pad 2: Net-(BT11-Pad2) -> Net-(BT107-Pad2)
- BT72 pad 1: Net-(BT11-Pad2) -> Net-(BT107-Pad2)
- BT72 pad 2: Net-(BT12-Pad2) -> Net-(BT108-Pad2)
- BT82 pad 1: Net-(BT1-Pad1) -> Net-(BT10-Pad1)
- BT82 pad 2: Net-(BT1-Pad2) -> Net-(BT10-Pad2)
- BT83 pad 1: Net-(BT1-Pad2) -> Net-(BT10-Pad2)
- BT83 pad 2: Net-(BT11-Pad2) -> Net-(BT107-Pad2)
- BT84 pad 1: Net-(BT11-Pad2) -> Net-(BT107-Pad2)
- BT84 pad 2: Net-(BT12-Pad2) -> Net-(BT108-Pad2)
- BT94 pad 1: Net-(BT1-Pad1) -> Net-(BT10-Pad1)
- BT94 pad 2: Net-(BT1-Pad2) -> Net-(BT10-Pad2)
- BT95 pad 1: Net-(BT1-Pad2) -> Net-(BT10-Pad2)
- BT95 pad 2: Net-(BT11-Pad2) -> Net-(BT107-Pad2)
- BT96 pad 1: Net-(BT11-Pad2) -> Net-(BT107-Pad2)
- BT96 pad 2: Net-(BT12-Pad2) -> Net-(BT108-Pad2)
- J1 pad 1: Net-(BT1-Pad1) -> Net-(BT108-Pad2)
- J2 pad 1: Net-(BT1-Pad2) -> Net-(J2-Pad1)
- J3 pad 1: Net-(BT11-Pad2) -> Net-(BT1-Pad1)
- TH1 pad 1: Net-(J7-Pad1) -> Net-(J2-Pad1)
- TH1 pad 2: Net-(J7-Pad2) -> Net-(J2-Pad2)
- TH2 pad 1: Net-(J9-Pad1) -> Net-(J2-Pad3)
- TH2 pad 2: Net-(J9-Pad2) -> Net-(J2-Pad4)
- TH3 pad 1: Net-(J8-Pad1) -> Net-(J2-Pad5)
- TH3 pad 2: Net-(J8-Pad2) -> Net-(J2-Pad6)
Routing:
- net Net-(BT108-Pad2): track 0.00 -> 488.5 mm
- net Net-(BT107-Pad2): track 0.00 -> 467.9 mm
- net Net-(BT10-Pad2): track 0.00 -> 433.5 mm
- net Net-(BT10-Pad1): track 0.00 -> 393.3 mm
- net Net-(BT1-Pad2): track 0.00 -> 383.7 mm, vias 200 -> 0
- net Net-(BT1-Pad1): track 0.00 -> 372.0 mm
- net Net-(BT110-Pad2): track 0.00 -> 360.3 mm
- net Net-(BT104-Pad2): track 0.00 -> 359.3 mm
- net Net-(BT103-Pad2): track 0.00 -> 318.0 mm
- net Net-(BT100-Pad1): track 0.00 -> 308.5 mm
- net Net-(BT102-Pad2): track 0.00 -> 304.4 mm
- net Net-(BT100-Pad2): track 0.00 -> 295.0 mm
- net Net-(BT101-Pad2): track 0.00 -> 285.8 mm
- net Net-(J2-Pad9): track 0.00 -> 212.6 mm, vias 0 -> 1
- net Net-(J2-Pad10): track 0.00 -> 209.3 mm, vias 0 -> 1
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- removed copper zone on B.Cu, net Net-(BT1-Pad1)
- removed copper zone on B.Cu, net Net-(BT1-Pad2)
- removed copper zone on F.Cu, net Net-(BT1-Pad2)
- removed copper zone on B.Cu, net Net-(BT11-Pad2)
- removed copper zone on F.Cu, net Net-(BT11-Pad2)
- removed copper zone on F.Cu, net Net-(BT12-Pad2)
Other:
- board size 100 x 100 mm -> 250 x 199 mm
- board text removed: "C0 C3 C6 C9 C12 C15"
- board text removed: "C1 C4 C7 C10 C13 C16"
- board text removed: "C12"
- board text removed: "C18"
- board text removed: "C2 C5 C8 C11 C14 C17"
- board text removed: "ENNOID"
- board text removed: "https://github.com/EnnoidMe/ENNOID-PACK"

Commit message: small changes to top pcb
Routing:
- net Net-(BT102-Pad2): track 304.4 -> 297.7 mm
- net Net-(BT108-Pad2): track 488.5 -> 493.2 mm
- net Net-(BT107-Pad2): track 467.9 -> 471.0 mm
- net Net-(BT103-Pad2): track 318.0 -> 314.9 mm
- net Net-(BT10-Pad2): track 433.5 -> 435.0 mm
- net Net-(BT104-Pad2): track 359.3 -> 357.8 mm

Commit message: Minor changes
Parts:
- added C1: 1u, Capacitors_SMD:C_0603_HandSoldering, F.Cu at (121.1, 189.7)
- added C10: 1u, Capacitors_SMD:C_0603_HandSoldering, F.Cu at (106.2, 183.8)
- added C11: 100n, Capacitors_SMD:C_0603_HandSoldering, F.Cu at (102.4, 182.4)
- added C12: 1u, Capacitors_SMD:C_0603_HandSoldering, F.Cu at (102.4, 183.8)
- added C2: 1u, Capacitors_SMD:C_0603_HandSoldering, F.Cu at (121.1, 188.1)
- added C3: 1u, Capacitors_SMD:C_0603_HandSoldering, F.Cu at (121.1, 186.5)
- added C4: 1u, Capacitors_SMD:C_0603_HandSoldering, F.Cu at (121.1, 184.8)
- added C5: 1u, Capacitors_SMD:C_0603_HandSoldering, F.Cu at (121.1, 183.3)
- added C6: 1u, Capacitors_SMD:C_0603_HandSoldering, F.Cu at (121.1, 181.7)
- added C7: 1u, Capacitors_SMD:C_0603_HandSoldering, F.Cu at (121.1, 180.1)
- added C8: 1u, Capacitors_SMD:C_0603_HandSoldering, F.Cu at (121.1, 178.5)
- added C9: 100n, Capacitors_SMD:C_0603_HandSoldering, F.Cu at (106.2, 182.4)
- added J4: Conn_01x04, Pin_Headers:Pin_Header_Straight_1x04_Pitch2.54mm, F.Cu at (102.0, 188.0)
- added R1: 100k, Resistors_SMD:R_0603_HandSoldering, F.Cu at (113.5, 189.7)
- added R10: 100k, Resistors_SMD:R_0603_HandSoldering, F.Cu at (106.4, 185.3)
- added R2: 100k, Resistors_SMD:R_0603_HandSoldering, F.Cu at (113.5, 188.1)
- added R3: 100k, Resistors_SMD:R_0603_HandSoldering, F.Cu at (113.5, 186.5)
- added R4: 100k, Resistors_SMD:R_0603_HandSoldering, F.Cu at (113.5, 184.9)
- added R5: 100k, Resistors_SMD:R_0603_HandSoldering, F.Cu at (113.5, 183.3)
- added R6: 100k, Resistors_SMD:R_0603_HandSoldering, F.Cu at (113.5, 181.7)
- added R7: 100k, Resistors_SMD:R_0603_HandSoldering, F.Cu at (113.5, 180.1)
- added R8: 100k, Resistors_SMD:R_0603_HandSoldering, F.Cu at (113.5, 178.5)
- added R9: 240, Resistors_SMD:R_0603_HandSoldering, F.Cu at (102.2, 185.3)
- added TH6: Thermistor, Resistors_SMD:R_0805_HandSoldering, F.Cu at (176.2, 54.6)
- added TH7: Thermistor, Resistors_SMD:R_0805_HandSoldering, F.Cu at (206.9, 37.8)
- added TH8: Thermistor, Resistors_SMD:R_0805_HandSoldering, F.Cu at (226.6, 15.0)
- added U1: ADC128D818, Housings_SSOP:TSSOP-16_4.4x5mm_Pitch0.65mm, F.Cu at (105.2, 177.7)
- J2: value Conn_01x10 -> Conn_01x04; footprint Pin_Headers:Pin_Header_Straight_1x10_Pitch2.54mm -> Connectors_Molex:Molex_KK-6410-04_04x2.54mm_Straight
- J3: footprint Pin_Headers:Pin_Header_Straight_1x13_Pitch2.54mm -> Connectors_Molex:Molex_KK-6410-13_13x2.54mm_Straight
- moved J3 186.5 mm to (157.5, 182.5), turned to 180 degrees
- moved TH5 70.7 mm to (147.0, 71.8)
- moved TH4 54.2 mm to (117.1, 90.3), turned to 180 degrees
- moved TH3 35.4 mm to (87.3, 107.2)
- moved TH2 19.8 mm to (56.7, 122.6)
- moved J2 13.9 mm to (84.1, 188.0), turned to 0 degrees
- moved J14 0.12 mm to (250.0, 87.1)
Connections:
- J2 pad 1: Net-(J2-Pad1) -> +5V
- J2 pad 4: Net-(J2-Pad4) -> GND
- TH1 pad 1: Net-(J2-Pad1) -> Net-(TH1-Pad1)
- TH1 pad 2: Net-(J2-Pad2) -> Net-(C8-Pad1)
- TH2 pad 1: Net-(J2-Pad3) -> Net-(TH2-Pad1)
- TH2 pad 2: Net-(J2-Pad4) -> Net-(C7-Pad1)
- TH3 pad 1: Net-(J2-Pad5) -> Net-(TH3-Pad1)
- TH3 pad 2: Net-(J2-Pad6) -> Net-(C6-Pad1)
- TH4 pad 1: Net-(J2-Pad7) -> Net-(TH4-Pad1)
- TH4 pad 2: Net-(J2-Pad8) -> Net-(C5-Pad1)
- TH5 pad 1: Net-(J2-Pad9) -> Net-(TH5-Pad1)
- TH5 pad 2: Net-(J2-Pad10) -> Net-(C4-Pad1)
Routing:
- net Net-(C1-Pad1): track 0.00 -> 270.2 mm, vias 0 -> 2
- net Net-(TH8-Pad1): track 0.00 -> 261.4 mm, vias 0 -> 2
- net Net-(C2-Pad1): track 0.00 -> 218.0 mm, vias 0 -> 2
- net Net-(TH7-Pad1): track 0.00 -> 213.3 mm, vias 0 -> 2
- net Net-(J2-Pad9): track 212.6 -> 0.00 mm, vias 1 -> 0
- net Net-(J2-Pad10): track 209.3 -> 0.00 mm, vias 1 -> 0
- net Net-(C3-Pad1): track 0.00 -> 177.9 mm, vias 0 -> 2
- net Net-(TH6-Pad1): track 0.00 -> 172.3 mm, vias 0 -> 2
- net Net-(J2-Pad7): track 154.6 -> 0.00 mm, vias 1 -> 0
- net Net-(J2-Pad8): track 153.3 -> 0.00 mm, vias 1 -> 0
- net Net-(C4-Pad1): track 0.00 -> 140.8 mm, vias 0 -> 2
- net Net-(TH5-Pad1): track 0.00 -> 135.1 mm, vias 0 -> 2
- net Net-(C8-Pad1): track 0.00 -> 122.3 mm, vias 0 -> 2
- net Net-(J2-Pad5): track 120.3 -> 0.00 mm, vias 1 -> 0
- net Net-(J2-Pad6): track 120.1 -> 0.00 mm, vias 1 -> 0
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- added copper zone on F.Cu, net +5V
- added copper zone on B.Cu, net GND
Other:
- board size 250 x 199 mm -> 250 x 192 mm

Commit message: readme
Parts:
- moved TH4 4.53 mm to (117.1, 85.8)
- moved TH8 2.96 mm to (226.1, 17.9)
- moved TH7 2.93 mm to (206.9, 34.9)
- moved TH6 2.52 mm to (176.2, 52.1)
- moved TH5 2.22 mm to (147.0, 69.5)
- moved TH3 2.10 mm to (87.3, 105.1)
- moved TH2 1.27 mm to (56.7, 121.3)
Routing:
- net Net-(BT107-Pad2): track 373.2 -> 433.7 mm
- net Net-(BT1-Pad1): track 320.1 -> 373.9 mm
- net Net-(BT100-Pad1): track 282.9 -> 327.4 mm
- net Net-(BT103-Pad2): track 296.5 -> 337.0 mm
- net Net-(BT10-Pad1): track 339.3 -> 374.8 mm
- net Net-(BT104-Pad2): track 319.9 -> 351.4 mm
- net Net-(BT102-Pad2): track 296.9 -> 328.4 mm
- net Net-(BT10-Pad2): track 360.1 -> 391.6 mm
- net Net-(BT1-Pad2): track 321.8 -> 353.3 mm
- net Net-(BT110-Pad2): track 313.6 -> 340.6 mm
- net Net-(BT100-Pad2): track 278.0 -> 305.0 mm
- net Net-(BT101-Pad2): track 274.0 -> 296.5 mm
- net Net-(TH4-Pad1): track 112.3 -> 116.8 mm
- net Net-(C5-Pad1): track 115.8 -> 120.3 mm
- net Net-(C2-Pad1): track 218.0 -> 220.9 mm
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
Commit message: Updated design
Parts:
- moved TH1 15.3 mm to (25.8, 155.0)
- moved TH7 15.3 mm to (191.7, 37.3)
- moved TH5 13.9 mm to (133.2, 71.3)
- moved TH6 13.9 mm to (162.5, 54.3)
- moved TH4 13.3 mm to (104.1, 88.2), turned to 0 degrees
- moved TH2 11.3 mm to (45.4, 121.8)
- moved U1 7.13 mm to (98.2, 179.0), turned to 180 degrees
- moved TH3 6.78 mm to (94.0, 105.1)
- moved R10 6.24 mm to (104.3, 179.5), turned to 90 degrees
- moved BT109 6.10 mm to (225.2, 161.2)
- moved BT97 6.04 mm to (235.0, 144.3)
- moved TH8 5.87 mm to (220.9, 20.5)
- moved BT110 5.72 mm to (205.8, 161.2)
- moved BT98 5.64 mm to (215.5, 144.3)
- moved BT73 5.60 mm to (235.0, 110.5)
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Routing:
- net Net-(BT1-Pad1): track 373.9 -> 95.7 mm
- net Net-(BT108-Pad2): track 375.3 -> 221.8 mm
- net Net-(BT100-Pad1): track 327.4 -> 226.8 mm
- net Net-(BT110-Pad2): track 340.6 -> 242.7 mm
- net Net-(BT102-Pad2): track 328.4 -> 231.0 mm
- net Net-(BT1-Pad2): track 353.3 -> 259.2 mm
- net Net-(BT100-Pad2): track 305.0 -> 212.8 mm
- net Net-(BT10-Pad1): track 374.8 -> 283.4 mm
- net Net-(BT10-Pad2): track 391.6 -> 304.8 mm
- net Net-(BT103-Pad2): track 337.0 -> 252.3 mm
- net Net-(BT104-Pad2): track 351.4 -> 268.0 mm
- net Net-(BT101-Pad2): track 296.5 -> 214.9 mm
- net Net-(BT107-Pad2): track 433.7 -> 368.0 mm
- net Net-(TH8-Pad1): track 260.3 -> 310.5 mm
- net Net-(TH6-Pad1): track 174.8 -> 209.7 mm
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Other:
- board size 250 x 192 mm -> 246 x 188 mm
